File: openkeebs.kicad_sch (KiCad schematic)
At the start: 0 parts

Commit message: add keys!
Parts:
- added D1, D10, D11, D12, D13, D14, D15, D16, D17, D18, D19, D2, D20, D21, D22, D23, D24, D25, D26, D27, D28, D29, D3, D30, D31, D32, D33, D34, D35, D36, D37, D38, D39, D4, D40, D41, D42, D43, D44, D45, D46, D47, D48, D49, D5, D50, D51, D52, D53, D54, D55, D56, D57, D58, D59, D6, D60, D61, D62, D63, D64, D65, D66, D67, D68, D69, D7, D70, D8, D9: Diode, symbol ScottoKeebs:Placeholder_Diode
- added S1, S10, S11, S12, S13, S14, S15, S16, S17, S18, S19, S2, S20, S21, S22, S23, S24, S25, S26, S27, S28, S29, S3, S30, S31, S32, S33, S34, S35, S36, S37, S38, S39, S4, S40, S41, S42, S43, S44, S45, S46, S47, S48, S49, S5, S50, S51, S52, S53, S54, S55, S56, S57, S58, S59, S6, S60, S61, S62, S63, S64, S65, S66, S67, S68, S69, S7, S70, S8, S9: Keyswitch, symbol ScottoKeebs:Placeholder_Keyswitch
Connections:
- new net: D33.2 (A), S33.2
- new net: D52.2 (A), S52.2
- new net: D53.2 (A), S53.2
- new net: D37.2 (A), S37.2
- new net: D38.2 (A), S38.2
- new net: D5.2 (A), S5.2
- new net: D29.2 (A), S29.2
- new net: D30.2 (A), S30.2
- new net: D68.2 (A), S68.2
- new net: D10.2 (A), S10.2
- new net: D12.2 (A), S12.2
- new net: D34.2 (A), S34.2
- new net: D59.2 (A), S59.2
- new net: D61.2 (A), S61.2
- new net: D4.2 (A), S4.2
- new net: D24.2 (A), S24.2
- new net: D17.2 (A), S17.2
- new net: D8.2 (A), S8.2
- new net: D16.2 (A), S16.2
- new net: D42.2 (A), S42.2
- new net: D1.2 (A), S1.2
- new net: D11.2 (A), S11.2
- new net: D48.2 (A), S48.2
- new net: D70.2 (A), S70.2
- new net: D9.2 (A), S9.2
- new net: D56.2 (A), S56.2
- new net: D22.2 (A), S22.2
- new net: D20.2 (A), S20.2
- new net: D14.2 (A), S14.2
- new net: D3.2 (A), S3.2
- new net: D69.2 (A), S69.2
- new net: D26.2 (A), S26.2
- new net: D23.2 (A), S23.2
- new net: D55.2 (A), S55.2
- new net: D36.2 (A), S36.2
- new net: D43.2 (A), S43.2
- new net: D50.2 (A), S50.2
- new net: D51.2 (A), S51.2
- new net: D27.2 (A), S27.2
- new net: D41.2 (A), S41.2
- new net: D2.2 (A), S2.2
- new net: D44.2 (A), S44.2
- new net: D6.2 (A), S6.2
- new net: D47.2 (A), S47.2
- new net: D13.2 (A), S13.2
- new net: D32.2 (A), S32.2
- new net: D7.2 (A), S7.2
- new net: D63.2 (A), S63.2
- new net: D28.2 (A), S28.2
- new net: D49.2 (A), S49.2
- new net: D40.2 (A), S40.2
- new net: D67.2 (A), S67.2
- new net: D39.2 (A), S39.2
- new net: D19.2 (A), S19.2
- new net: D25.2 (A), S25.2
- new net: D15.2 (A), S15.2
- new net: D18.2 (A), S18.2
- new net: D54.2 (A), S54.2
- new net: D65.2 (A), S65.2
- new net: D58.2 (A), S58.2
- new net: D60.2 (A), S60.2
- new net: D35.2 (A), S35.2
- new net: D31.2 (A), S31.2
- new net: D62.2 (A), S62.2
- new net: D64.2 (A), S64.2
- new net: D66.2 (A), S66.2
- new net: D57.2 (A), S57.2
- new net: D21.2 (A), S21.2
- new net: D45.2 (A), S45.2
- new net: D46.2 (A), S46.2
